Commit message: Fix quadrotor xacro XML structure (close gazebo tag and xacro:macro properly)

File: src/robots/quadrotor_sitl/urdf/quadrotor_gazebo.xacro (robot description, xacro)
@@ -95,5 +95,5 @@
         </plugin>
       </xacro:if>
-    </plugin>
-  </gazebo>
+    </gazebo>
+  </xacro:macro>
 </robot>
