Commit message: mujoco fix

File: src/robot_lab_robots/berkeley_humanoid_lite/urdf/berkeley_humanoid_lite_biped.urdf (robot description, URDF)
Before this commit: robot berkeley-humanoid-lite, 15 links, 14 joints
Links:
- link base: geometry collision box size=0.15 0.14 0.23; visual mesh filename=package://robot_lab_robots/berkeley_humanoid_lite/meshes/ba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
- link imu_2: geometry visual mesh filename=package://robot_lab_robots/berkeley_humanoid_lite/meshes/im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
- link leg_left_ankle_pitch: geometry visual mesh filename=package://robot_lab_robots/berkeley_humanoid_lite/meshes/le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
- link leg_left_ankle_roll: geometry collision box size=0.072 0.22 0.04; visual mesh filename=package://robot_lab_robots/berkeley_humanoid_lite/meshes/le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
- link leg_left_hip_pitch: geometry collision cylinder length=0.13 radius=0.05; visual mesh filename=package://robot_lab_robots/berkeley_humanoid_lite/meshes/le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
- link leg_left_hip_roll: geometry visual mesh filename=package://robot_lab_robots/berkeley_humanoid_lite/meshes/le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
- link leg_left_hip_yaw: geometry visual mesh filename=package://robot_lab_robots/berkeley_humanoid_lite/meshes/le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
- link leg_left_knee_pitch: geometry collision cylinder length=0.15 radius=0.04; visual mesh filename=package://robot_lab_robots/berkeley_humanoid_lite/meshes/le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
- link leg_right_ankle_pitch: geometry visual mesh filename=package://robot_lab_robots/berkeley_humanoid_lite/meshes/le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
- link leg_right_ankle_roll: geometry collision box size=0.072 0.22 0.04; visual mesh filename=package://robot_lab_robots/berkeley_humanoid_lite/meshes/le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
- link leg_right_hip_pitch: geometry collision cylinder length=0.13 radius=0.05; visual mesh filename=package://robot_lab_robots/berkeley_humanoid_lite/meshes/le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
- link leg_right_hip_roll: geometry visual mesh filename=package://robot_lab_robots/berkeley_humanoid_lite/meshes/le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
- link leg_right_hip_yaw: geometry visual mesh filename=package://robot_lab_robots/berkeley_humanoid_lite/meshes/le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
- link leg_right_knee_pitch: geometry collision cylinder length=0.15 radius=0.04; visual mesh filename=package://robot_lab_robots/berkeley_humanoid_lite/meshes/le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

File: src/robot_lab_robots/unitree/b2_description_mujoco/xml/b2_description.urdf (robot description, URDF)
Before this commit: robot b2_description, 44 links, 43 joints
Links:
- link FL_thigh_protect: geometry visual mesh filename=package://robot_lab_robots/unitree/b2_description_mujoco/me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
- link FR_foot: geometry collision cylinder length=0.05 radius=0.032; visual mesh filename=package://robot_lab_robots/unitree/b2_description_mujoco/me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
- link FR_thigh_protect: geometry visual mesh filename=package://robot_lab_robots/unitree/b2_description_mujoco/me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
- link RL_foot: geometry collision cylinder length=0.05 radius=0.032; visual mesh filename=package://robot_lab_robots/unitree/b2_description_mujoco/me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
- link RL_thigh_protect: geometry visual mesh filename=package://robot_lab_robots/unitree/b2_description_mujoco/me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
- link RR_foot: geometry collision cylinder length=0.05 radius=0.032; visual mesh filename=package://robot_lab_robots/unitree/b2_description_mujoco/me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
- link RR_thigh_protect: geometry visual mesh filename=package://robot_lab_robots/unitree/b2_description_mujoco/me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
- link f_dc_link: geometry visual mesh filename=package://robot_lab_robots/unitree/b2_description_mujoco/me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
- link f_oc_link: geometry visual mesh filename=package://robot_lab_robots/unitree/b2_description_mujoco/me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
- link head_Link: geometry collision box size=0.04 0.12 0.14; visual mesh filename=package://robot_lab_robots/unitree/b2_description_mujoco/me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
- link imu_link: geometry visual mesh filename=package://robot_lab_robots/unitree/b2_description_mujoco/me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
- link lidar_link: geometry collision cylinder length=0.16 radius=0.076; visual mesh filename=package://robot_lab_robots/unitree/b2_description_mujoco/me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
- link logo_left_link: geometry visual mesh filename=package://robot_lab_robots/unitree/b2_description_mujoco/me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
- link logo_right_link: geometry visual mesh filename=package://robot_lab_robots/unitree/b2_description_mujoco/me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
- link r_dc_link: geometry visual mesh filename=package://robot_lab_robots/unitree/b2_description_mujoco/me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
- link r_oc_link: geometry visual mesh filename=package://robot_lab_robots/unitree/b2_description_mujoco/me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
- link tail_link: geometry collision box size=0.025 0.12 0.14; visual mesh filename=package://robot_lab_robots/unitree/b2_description_mujoco/me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
