Commit message: fix(bhl): rename colliding imu joint for Gazebo SDF spawn

File: src/robot_lab_robots/berkeley_humanoid_lite/urdf/berkeley_humanoid_lite.urdf (robot description, URDF)
Before this commit: robot berkeley-humanoid-lite, 27 links, 26 joints
Joints:
- removed joint imu
- added joint imu_mount_joint: type fixed, parent base, child imu_2, origin xyz=0.061722 -5.97549e-17 0.68 rpy=-6.12323e-17 1.13243e-14 -1.20616e-15, axis 0 0 1, limit effort=20 velocity=15

File: src/robot_lab_robots/berkeley_humanoid_lite/urdf/berkeley_humanoid_lite_biped.urdf (robot description, URDF)
Before this commit: robot berkeley-humanoid-lite, 15 links, 14 joints
Joints:
- removed joint imu
- added joint imu_mount_joint: type fixed, parent base, child imu_2, origin xyz=0.061722 -1.49319e-16 0.68 rpy=-6.12323e-17 2.26485e-14 -2.65724e-15, axis 0 0 1, limit effort=20 velocity=15
