Commit message: feat(sim): raise spawned robot height for Gazebo and add partition reaper
Add helper functions to detect ros2_control blocks and compute a
spawn height that keeps the robot's lowest collision point above the
floor (based on the xacro-generated URDF), then use it for non-free
Gazebo spawns. This prevents robots from being buried in the ground
since Gazebo spawns blindly unlike the other backends that lift from
their collision bounds.

Also launch a detached partition_reaper process alongside Gazebo
simulations to clean up the Gazebo server which can outlive the launch.

Update _build_simulation_actions to use the cleared spawn height and
the reaper for Gazebo spawns, and restructure the display logic to
always spawn non-free robots into the world (removed the special
joint-slider preview-only case for free robots).

File: src/robot_lab_robots/labbot/urdf/labbot.urdf.xacro (robot description, xacro)
@@ -98,4 +98,7 @@
     <axis xyz="0 1 0"/>
   </joint>
+  <!-- Two passive casters, front and rear, so the drive wheels at the
+       base centre are not the only support along the fore-aft axis:
+       with one caster the body could pitch onto its unsupported end. -->
   <!-- Rear passive caster: sphere radius 0.03 m -->
   <link name="caster_rear_link">
@@ -124,4 +127,30 @@
     <origin xyz="-0.12 0 -0.09" rpy="0 0 0"/>
   </joint>
+  <!-- Front passive caster: sphere radius 0.03 m -->
+  <link name="caster_front_link">
+    <inertial>
+      <origin xyz="0 0 0" rpy="0 0 0"/>
+      <mass value="0.05"/>
+      <inertia ixx="1.8e-5" ixy="0" ixz="0" iyy="1.8e-5" iyz="0" izz="1.8e-5"/>
+    </inertial>
+    <visual>
+      <origin xyz="0 0 0" rpy="0 0 0"/>
+      <geometry>
+        <sphere radius="0.03"/>
+      </geometry>
+      <material name="labbot_black"/>
+    </visual>
+    <collision>
+      <origin xyz="0 0 0" rpy="0 0 0"/>
+      <geometry>
+        <sphere radius="0.03"/>
+      </geometry>
+    </collision>
+  </link>
+  <joint name="caster_front_joint" type="fixed">
+    <parent link="base_link"/>
+    <child link="caster_front_link"/>
+    <origin xyz="0.12 0 -0.09" rpy="0 0 0"/>
+  </joint>
   <!-- IMU -->
   <link name="imu_link">
@@ -176,4 +205,9 @@
     <origin xyz="0 0 0.08" rpy="0 0 0"/>
   </joint>
+  <!-- Used by the shared OAK-D macro, which expects the including robot
+       to define it (Bumperbot does). -->
+  <material name="dark_grey">
+    <color rgba="0.3 0.3 0.3 1"/>
+  </material>
   <material name="labbot_grey">
     <color rgba="0.5 0.5 0.5 1"/>

File: src/robot_lab_robots/labbot/urdf/labbot_gazebo.xacro (robot description, xacro)
@@ -20,6 +20,14 @@
     <fdir1>1 0 0</fdir1>
   </gazebo>
-  <!-- Caster Wheel -->
+  <!-- Caster Wheels -->
   <gazebo reference="caster_rear_link">
+    <mu1>0.1</mu1>
+    <mu2>0.1</mu2>
+    <kp>1000000.0</kp>
+    <kd>100.0</kd>
+    <minDepth>0.001</minDepth>
+    <maxVel>1.0</maxVel>
+  </gazebo>
+  <gazebo reference="caster_front_link">
     <mu1>0.1</mu1>
     <mu2>0.1</mu2>
