Commit message: git hub coilot + misterl vibe + cline with deep seek and super bunny alpha worked on R5, R6 and R7

File: src/robot_lab_robots/ackermann_car/urdf/ackermann_car_macro.xacro (robot description, xacro)
@@ -68,7 +68,15 @@
       </visual>
       <collision>
+        <!-- Wheel wells: the chassis collision is narrower than the body
+             shell (0.16 m vs 0.22 m).  At the full steering swing the
+             tire's inner rim reaches y = min(0.14 - 0.02*cos(0.8) -
+             0.05*sin(0.8)) = 0.090 m, and a full-width collision box
+             (edge at 0.11 m) made MuJoCo resolve the sweep with a ~113 N
+             chassis-tire contact that saturated the 10 N*m steering
+             servos (0.23 rad measured of 0.45 commanded, 2026-10-01).
+             The visual keeps the full shell. -->
         <origin xyz="${body_x} 0 0.04" rpy="0 0 0"/>
         <geometry>
-          <box size="0.48 0.22 0.08"/>
+          <box size="0.48 0.16 0.08"/>
         </geometry>
       </collision>

File: src/robot_lab_robots/holonomic_wheels/urdf/holonomic_wheels_macro.xacro (robot description, xacro)
@@ -103,7 +103,13 @@
       </visual>
       <collision>
+        <!-- Wheel wells: the chassis collision is narrower than the body
+             shell (0.20 m vs 0.30 m) so the steered wheels' swept volume
+             clears it.  At the 0.785 rad steering limit a 0.05 m wheel at
+             y=0.16 reaches min y = 0.16 - 0.02*cos(0.785) -
+             0.05*sin(0.785) = 0.110 m; a full-width box (edge 0.15 m)
+             overlapped even the rest pose.  The visual keeps the shell. -->
         <origin xyz="0 0 0.04" rpy="0 0 0"/>
         <geometry>
-          <box size="0.46 0.30 0.08"/>
+          <box size="0.46 0.20 0.08"/>
         </geometry>
       </collision>
