Commit message: R5.6: verify four-wheel motion and expose mecanum gaps

File: src/robot_lab_robots/holonomic_wheels/urdf/holonomic_wheels_macro.xacro (robot description, xacro)
@@ -54,5 +54,5 @@
   <!-- One steered wheel: a knuckle link carries the wheel, so the wheel can
        spin about its own axis while the knuckle aims it. -->
-  <xacro:macro name="steerable_wheel" params="corner">
+  <xacro:macro name="steerable_wheel" params="corner x y">
     <link name="${corner}_steer_link">
       <inertial>
@@ -71,5 +71,5 @@
       <parent link="base_link"/>
       <child link="${corner}_steer_link"/>
-      <origin xyz="0 0 0" rpy="0 0 0"/>
+      <origin xyz="${x} ${y} 0" rpy="0 0 0"/>
       <axis xyz="0 0 1"/>
       <limit lower="-0.785" upper="0.785" effort="10.0" velocity="3.0"/>
@@ -80,5 +80,5 @@
       <parent link="${corner}_steer_link"/>
       <child link="${corner}_wheel_link"/>
-      <origin xyz="0 0 -0.038" rpy="0 0 0"/>
+      <origin xyz="0 0 -0.012" rpy="0 0 0"/>
       <axis xyz="0 1 0"/>
       <dynamics damping="0.005" friction="0.0"/>
@@ -238,8 +238,8 @@
     <xacro:holonomic_chassis robot_name="${robot_name}"/>
     <xacro:holonomic_sensors/>
-    <xacro:steerable_wheel corner="front_left"/>
-    <xacro:steerable_wheel corner="front_right"/>
-    <xacro:steerable_wheel corner="rear_left"/>
-    <xacro:steerable_wheel corner="rear_right"/>
+    <xacro:steerable_wheel corner="front_left" x="0.16" y="0.16"/>
+    <xacro:steerable_wheel corner="front_right" x="0.16" y="-0.16"/>
+    <xacro:steerable_wheel corner="rear_left" x="-0.16" y="0.16"/>
+    <xacro:steerable_wheel corner="rear_right" x="-0.16" y="-0.16"/>
     <xacro:holonomic_control steer="true"/>
     <xacro:holonomic_gazebo robot_name="${robot_name}"/>

Commit message: codex work

File: src/robot_lab_robots/holonomic_wheels/urdf/holonomic_wheels_macro.xacro (robot description, xacro)
@@ -23,4 +23,5 @@
 -->
 <robot xmlns:xacro="http://www.ros.org/wiki/xacro">
+  <xacro:include filename="$(find robot_lab_robots)/holonomic_wheels/urdf/mecanum_rollers.xacro"/>
   <xacro:macro name="holonomic_wheel" params="name radius:=0.05 width:=0.04 mass:=0.3">
     <link name="${name}_link">
@@ -141,5 +142,10 @@
     <ros2_control name="GazeboSimSystem" type="system">
       <hardware>
-        <plugin>gz_ros2_control/GazeboSimROS2ControlPlugin</plugin>
+        <xacro:if value="$(arg is_ignition)">
+          <plugin>ign_ros2_control/IgnitionSystem</plugin>
+        </xacro:if>
+        <xacro:unless value="$(arg is_ignition)">
+          <plugin>gz_ros2_control/GazeboSimSystem</plugin>
+        </xacro:unless>
       </hardware>
       <xacro:if value="${steer}">
@@ -249,37 +255,8 @@
     <xacro:holonomic_chassis robot_name="${robot_name}"/>
     <xacro:holonomic_sensors/>
-    <!-- Fixed wheels: four drive joints and no steering joints at all. -->
-    <xacro:holonomic_wheel name="front_left_wheel"/>
-    <joint name="front_left_wheel_joint" type="continuous">
-      <parent link="base_link"/>
-      <child link="front_left_wheel_link"/>
-      <origin xyz="0.16 0.16 -0.012" rpy="0 0 0"/>
-      <axis xyz="0 1 0"/>
-      <dynamics damping="0.005" friction="0.0"/>
-    </joint>
-    <xacro:holonomic_wheel name="front_right_wheel"/>
-    <joint name="front_right_wheel_joint" type="continuous">
-      <parent link="base_link"/>
-      <child link="front_right_wheel_link"/>
-      <origin xyz="0.16 -0.16 -0.012" rpy="0 0 0"/>
-      <axis xyz="0 1 0"/>
-      <dynamics damping="0.005" friction="0.0"/>
-    </joint>
-    <xacro:holonomic_wheel name="rear_left_wheel"/>
-    <joint name="rear_left_wheel_joint" type="continuous">
-      <parent link="base_link"/>
-      <child link="rear_left_wheel_link"/>
-      <origin xyz="-0.16 0.16 -0.012" rpy="0 0 0"/>
-      <axis xyz="0 1 0"/>
-      <dynamics damping="0.005" friction="0.0"/>
-    </joint>
-    <xacro:holonomic_wheel name="rear_right_wheel"/>
-    <joint name="rear_right_wheel_joint" type="continuous">
-      <parent link="base_link"/>
-      <child link="rear_right_wheel_link"/>
-      <origin xyz="-0.16 -0.16 -0.012" rpy="0 0 0"/>
-      <axis xyz="0 1 0"/>
-      <dynamics damping="0.005" friction="0.0"/>
-    </joint>
+    <xacro:physical_mecanum_wheel corner="front_left" x="0.16" y="0.16" side="-1"/>
+    <xacro:physical_mecanum_wheel corner="front_right" x="0.16" y="-0.16" side="1"/>
+    <xacro:physical_mecanum_wheel corner="rear_left" x="-0.16" y="0.16" side="1"/>
+    <xacro:physical_mecanum_wheel corner="rear_right" x="-0.16" y="-0.16" side="-1"/>
     <xacro:holonomic_control steer="false"/>
     <xacro:holonomic_gazebo robot_name="${robot_name}"/>

Commit message: R5.4/R5.6: integrate PX4 flight and four-wheel navigation
Expose measured Flight services and faithful steering commands in Robot Lab GUI. Repair wheel rolling/pivot, physical mecanum collision cost, real Nav2/AMCL dispatch and Isaac lateral commands; preserve scoped live results and failed trials.

Include SSD relocation records, restored third-party notices, completion audit, existing verification-script moves, and updated roadmap/agent guides with the remaining qualification gaps.

File: src/robot_lab_robots/holonomic_wheels/urdf/holonomic_wheels_macro.xacro (robot description, xacro)
@@ -10,7 +10,6 @@
                      (robot_lab_utils/drive_kinematics.py), not a different
                      description: the same eight joints serve all four.
-  mecanum            four fixed wheels on 45-degree rollers.  The rollers are
-                     visual only and need no joint; the lateral freedom comes
-                     from their geometry, which the drive model inverts.
+  mecanum            four driven hubs with 60 passive physical rollers in
+                     an X layout. These joints must remain free in physics.
   base_footprint is the geometric centre on the ground.  For the two
   curvature-following 4WS patterns that is the point with no sideways velocity,
@@ -18,5 +17,5 @@
   across every wheeled robot here.
   Dimensions: wheelbase 0.32 m, track 0.32 m, wheel radius 0.05 m, body
-  0.46 x 0.30 x 0.08 m.  The 4WS steering limit is +/-0.785 rad (45 deg), which
+  0.46 x 0.30 x 0.08 m.  The 4WS steering limit is +/-1.5707963267948966 rad (45 deg), which
   at a 0.16 m half-wheelbase gives a 0.16 m minimum turning radius - far tighter
   than a car, which is the reason to run this base at all.
@@ -74,5 +73,5 @@
       <origin xyz="${x} ${y} 0" rpy="0 0 0"/>
       <axis xyz="0 0 1"/>
-      <limit lower="-0.785" upper="0.785" effort="10.0" velocity="3.0"/>
+      <limit lower="-1.5707963267948966" upper="1.5707963267948966" effort="10.0" velocity="3.0"/>
       <dynamics damping="0.05" friction="0.0"/>
     </joint>
@@ -105,7 +104,6 @@
         <!-- Wheel wells: the chassis collision is narrower than the body
              shell (0.20 m vs 0.30 m) so the steered wheels' swept volume
-             clears it.  At the 0.785 rad steering limit a 0.05 m wheel at
-             y=0.16 reaches min y = 0.16 - 0.02*cos(0.785) -
-             0.05*sin(0.785) = 0.110 m; a full-width box (edge 0.15 m)
+             clears it throughout +/-90 degrees. The wheel swept radius
+             is sqrt(0.05^2 + 0.02^2), leaving min y = 0.106 m; a full-width box (edge 0.15 m)
              overlapped even the rest pose.  The visual keeps the shell. -->
         <origin xyz="0 0 0.04" rpy="0 0 0"/>
@@ -122,4 +120,7 @@
   </xacro:macro>
   <xacro:macro name="holonomic_sensors">
+    <xacro:oakd parent_link="base_link" mesh_visual="false">
+      <origin xyz="0.20 0 0.13" rpy="0 0 0"/>
+    </xacro:oakd>
     <link name="imu_link">
       <inertial>
@@ -159,6 +160,6 @@
           <joint name="${joint}">
             <command_interface name="position">
-              <param name="min">-0.785</param>
-              <param name="max">0.785</param>
+              <param name="min">-1.5707963267948966</param>
+              <param name="max">1.5707963267948966</param>
             </command_interface>
             <state_interface name="position"/>
@@ -189,4 +190,25 @@
   <xacro:macro name="holonomic_gazebo" params="robot_name">
     <gazebo>
+      <!-- Independent model pose, never wheel odometry or a commanded pose. -->
+      <xacro:if value="$(arg is_ignition)">
+        <plugin filename="ignition-gazebo-odometry-publisher-system" name="ignition::gazebo::systems::OdometryPublisher">
+          <odom_frame>world</odom_frame>
+          <robot_base_frame>base_footprint</robot_base_frame>
+          <odom_topic>/model/${robot_name}/odometry_truth</odom_topic>
+          <tf_topic>/model/${robot_name}/truth_pose</tf_topic>
+          <dimensions>3</dimensions>
+          <odom_publish_frequency>50</odom_publish_frequency>
+        </plugin>
+      </xacro:if>
+      <xacro:unless value="$(arg is_ignition)">
+        <plugin filename="gz-sim-odometry-publisher-system" name="gz::sim::systems::OdometryPublisher">
+          <odom_frame>world</odom_frame>
+          <robot_base_frame>base_footprint</robot_base_frame>
+          <odom_topic>/model/${robot_name}/odometry_truth</odom_topic>
+          <tf_topic>/model/${robot_name}/truth_pose</tf_topic>
+          <dimensions>3</dimensions>
+          <odom_publish_frequency>50</odom_publish_frequency>
+        </plugin>
+      </xacro:unless>
       <xacro:if value="$(arg is_ignition)">
         <plugin filename="ign_ros2_control-system" name="ign_ros2_control::IgnitionROS2ControlPlugin">

File: src/robot_lab_robots/holonomic_wheels/urdf/mecanum_rollers.xacro (robot description, xacro)
@@ -13,5 +13,5 @@
         </visual>
         <collision>
-          <geometry><mesh filename="package://robot_lab_robots/holonomic_wheels/third_party/fuji_mecanum/roller.stl" scale="${mecanum_scale} ${mecanum_scale} ${mecanum_scale}"/></geometry>
+          <geometry><mesh filename="package://robot_lab_robots/holonomic_wheels/third_party/fuji_mecanum/roller_collision.stl" scale="${mecanum_scale} ${mecanum_scale} ${mecanum_scale}"/></geometry>
         </collision>
         <inertial>
