Commit message: Gazebo: run legged policies through an effort PD trajectory controller (Go2)
Go2 can now localize in Gazebo, completing the user's "BHL/Go2 localization
not offered in Gazebo/Isaac" request for Go2. In Gazebo localization the
robot's rl_sar policy is selected, as in Isaac, and legged_policy:=none
turns it off.

Its PD law tau = kp (q* - q) + kd (dq* - dq) runs in the description's
ros2_control at 500 Hz. The controller is a joint_trajectory_controller
with effort commands, loaded by the spawner with the policy gains:
legged_policy.ros2_control_pd_parameters. Its PID uses measured joint
velocity, so a target step causes no derivative spike.
legged-policy-controller also publishes each target set as a one-point
JointTrajectory. The wheeled controller layer is skipped.

The Go2 sim description gains a head LiDAR (laser_link, gpu_lidar
/scan). The Go2 profile declares ros2_control and lidar_2d, and
mode_capability gives Gazebo stance to legged_policy robots with a
ros2_control block.

Implemented and unit/launch-tested only. The native Gazebo trial is
queued.

Co-Authored-By: Claude Opus 5.5 <noreply@anthropic.com>

File: src/robot_lab_robots/unitree/go2_description/xacro/go2_sim.xacro (robot description, xacro)
@@ -12,3 +12,45 @@
   <xacro:include filename="$(find robot_lab_robots)/unitree/go2_description/xacro/go2_ros2_control.xacro"/>
   <xacro:go2_ros2_control is_ignition="$(arg is_ignition)"/>
+  <!-- 2D LiDAR for localization (2026-10-12), at the front of the trunk where
+       the real Go2 carries its head LiDAR, clear of the trunk and legs.  Gazebo renders
+       it; the PyBullet/MuJoCo/Isaac bridges cast their scan from this link. -->
+  <joint name="laser_joint" type="fixed">
+    <parent link="trunk"/>
+    <child link="laser_link"/>
+    <origin xyz="0.20 0 0.12" rpy="0 0 0"/>
+  </joint>
+  <link name="laser_link">
+    <inertial>
+      <mass value="0.01"/>
+      <inertia ixx="1e-6" ixy="0" ixz="0" iyy="1e-6" iyz="0" izz="1e-6"/>
+    </inertial>
+  </link>
+  <gazebo reference="laser_link">
+    <sensor name="lidar" type="gpu_lidar">
+      <always_on>true</always_on>
+      <topic>scan</topic>
+      <update_rate>5</update_rate>
+      <gz_frame_id>laser_link</gz_frame_id>
+      <lidar>
+        <scan>
+          <horizontal>
+            <samples>360</samples>
+            <resolution>1.0</resolution>
+            <min_angle>0.0</min_angle>
+            <max_angle>6.28</max_angle>
+          </horizontal>
+        </scan>
+        <range>
+          <min>0.12</min>
+          <max>12.0</max>
+          <resolution>0.02</resolution>
+        </range>
+        <noise>
+          <type>gaussian</type>
+          <mean>0.0</mean>
+          <stddev>0.01</stddev>
+        </noise>
+      </lidar>
+    </sensor>
+  </gazebo>
 </robot>
