Commit message: MOLAR: lift and telescope hard stops 5 mm below the controlled range
Fortress/DART's velocity servo, which gz_ros2_control uses for position
commands, cannot leave a position limit the joint rests on: the lift,
spawned on its lower stop under the 139 N carriage load, never rose for a
0.06 m command, while the unloaded telescope moved. With the derivative's
hard stops at -0.005 m (the articulation contract still bounds commands to
0-0.68 m and 0-0.14 m) the Gazebo lift reaches 0.06 m. Both variants; the
provisioner writes it; the source URDFs are unchanged.

Co-Authored-By: Claude Opus 5.5 <noreply@anthropic.com>

File: src/robot_lab_robots/molar_hri/urdf/molar_hri.urdf.xacro (robot description, xacro)
@@ -1205,5 +1205,5 @@
     <origin xyz="0.0005 0 0.42" rpy="0 0 0" />
     <axis xyz="0 0 1" />
-    <limit effort="2000" velocity="0.035" lower="0" upper="0.68" />
+    <limit effort="2000" velocity="0.035" lower="-0.005" upper="0.68" />
     <dynamics damping="30" friction="0" />
   </joint>
@@ -1213,5 +1213,5 @@
     <origin xyz="0 0 0" rpy="0 0 0" />
     <axis xyz="1 0 0" />
-    <limit effort="250" velocity="0.1" lower="0" upper="0.14" />
+    <limit effort="250" velocity="0.1" lower="-0.005" upper="0.14" />
     <dynamics damping="8" friction="0" />
   </joint>
@@ -1221,5 +1221,5 @@
     <origin xyz="0 0 0" rpy="0 0 0" />
     <axis xyz="1 0 0" />
-    <limit effort="250" velocity="0.1" lower="0" upper="0.14" />
+    <limit effort="250" velocity="0.1" lower="-0.005" upper="0.14" />
     <dynamics damping="8" friction="0" />
   </joint>

File: src/robot_lab_robots/probot_l/urdf/probot_l.urdf.xacro (robot description, xacro)
@@ -701,5 +701,5 @@
     <origin xyz="0.0005 0 0.42" rpy="0 0 0" />
     <axis xyz="0 0 1" />
-    <limit effort="2000" velocity="0.035" lower="0" upper="0.68" />
+    <limit effort="2000" velocity="0.035" lower="-0.005" upper="0.68" />
     <dynamics damping="30" friction="0" />
   </joint>
@@ -709,5 +709,5 @@
     <origin xyz="0 0 0" rpy="0 0 0" />
     <axis xyz="1 0 0" />
-    <limit effort="250" velocity="0.1" lower="0" upper="0.14" />
+    <limit effort="250" velocity="0.1" lower="-0.005" upper="0.14" />
     <dynamics damping="8" friction="0" />
   </joint>
@@ -717,5 +717,5 @@
     <origin xyz="0 0 0" rpy="0 0 0" />
     <axis xyz="1 0 0" />
-    <limit effort="250" velocity="0.1" lower="0" upper="0.14" />
+    <limit effort="250" velocity="0.1" lower="-0.005" upper="0.14" />
     <dynamics damping="8" friction="0" />
   </joint>
