Commit message: feat: connect GUI to common resolver for R3.4
Advance R3.3 to done and mark R3.4 (Connect GUI to the common resolver) as active. Adds headless GUI-adjacent composition logic (gui_composition.py) that builds resolver.ExperimentRequest from GuiCompositionSelection using the same resolver/validator as the CLI, serializing identical manifest YAML. Includes 11 headless tests verifying CLI/GUI manifest parity, profile reload, selection changes active nav2 plugin, validator rejection of invalid selections, and legacy profile migration. Extends scope to multiple robot_lab packages and adds robot config paths. Updates R3.4 next action to address 2026-09-22 user regression report on map-only and robot-plus-map display, humanoid stability, Labbot Gazebo spawn, and mobile SLAM/navigation launches. Also stabilizes humanoid policy controller ramp with stance PD gains and ankle-strategy tilt feedback from balance core.

File: src/robot_lab_robots/description_common/urdf/oakd_camera.xacro (robot description, xacro)
@@ -9,5 +9,5 @@
   </xacro:macro>
   <!-- Reusable OAK-D Pro / RGBD camera macro -->
-  <xacro:macro name="oakd" params="name:=oakd parent_link *origin model:=pro">
+  <xacro:macro name="oakd" params="name:=oakd parent_link *origin model:=pro mesh_visual:=true">
     <xacro:property name="baseline" value="0.075"/>
     <xacro:property name="oakd_pi" value="3.1415926535897931"/>
@@ -21,5 +21,10 @@
       <visual>
         <geometry>
-          <mesh filename="package://robot_lab_robots/description_common/meshes/oakd_${model}.stl" scale="1 1 1"/>
+          <xacro:if value="${mesh_visual}">
+            <mesh filename="package://robot_lab_robots/description_common/meshes/oakd_${model}.stl" scale="1 1 1"/>
+          </xacro:if>
+          <xacro:unless value="${mesh_visual}">
+            <box size="0.0225 0.097 0.03"/>
+          </xacro:unless>
         </geometry>
         <material name="dark_grey"/>

File: src/robot_lab_robots/labbot/urdf/labbot.urdf.xacro (robot description, xacro)
@@ -5,4 +5,8 @@
   <!-- Load Simulated or Real Hardware Interfaces -->
   <xacro:arg name="is_sim" default="true"/>
+  <xacro:include filename="$(find robot_lab_robots)/description_common/urdf/oakd_camera.xacro" />
+  <xacro:oakd name="oakd" parent_link="base_link" model="pro" mesh_visual="false">
+    <origin xyz="0.12 0 0.09" rpy="0 0 0"/>
+  </xacro:oakd>
   <!-- Include Gazebo Parameters -->
   <xacro:include filename="$(find robot_lab_robots)/labbot/urdf/labbot_gazebo.xacro" />

Commit message: feat: validate fleet workloads and update catalog restoration status
Add schema-aware validation for robot_lab.fleet_workload.v1 workloads in ConcurrentRunner, requiring the shared-world navigation launch, prevent per-member reset of fleet batches, and record workload schema on jobs. Update platform status to mark the seven missing robot registrations restored via cached source repairs.

File: src/robot_lab_robots/description_common/urdf/oakd_camera.xacro (robot description, xacro)
@@ -9,5 +9,5 @@
   </xacro:macro>
   <!-- Reusable OAK-D Pro / RGBD camera macro -->
-  <xacro:macro name="oakd" params="name:=oakd parent_link *origin model:=pro mesh_visual:=true">
+  <xacro:macro name="oakd" params="name:=oakd parent_link *origin model:=pro mesh_visual:=true rate:=30">
     <xacro:property name="baseline" value="0.075"/>
     <xacro:property name="oakd_pi" value="3.1415926535897931"/>
@@ -101,5 +101,5 @@
       <sensor name="rgbd_camera" type="rgbd_camera">
         <always_on>1</always_on>
-        <update_rate>30</update_rate>
+        <update_rate>${rate}</update_rate>
         <visualize>true</visualize>
         <camera>

File: src/robot_lab_robots/lab_rov/urdf/lab_rov.urdf.xacro (robot description, xacro)
@@ -28,5 +28,5 @@
     </collision>
   </link>
-  <xacro:oakd name="oakd" parent_link="base_link" model="pro" mesh_visual="false">
+  <xacro:oakd name="oakd" parent_link="base_link" model="pro" mesh_visual="false" rate="5">
     <origin xyz=".21 0 .06" rpy="0 0 0" />
   </xacro:oakd>
