Commit message: Conventional commit message:
feat: update docs and roadmap for October 27 native continuation delivery

Add notes on native marine/gait acquisition, navigation, range-reference formation, operator-loss landing, fleet batch reset, and tracked family workloads; update the roadmap and move the primary workflow record to docs/status/native-workflows-2026-10-27.md while preserving the earlier delivery as the catalog scope reference.

File: src/robot_lab_robots/lab_tracked/robot.urdf (robot description, URDF)
Before this commit: robot lab_tracked, 8 links, 7 joints
Joints:
- joint footprint_fixed: origin (none) -> xyz=0 0 .07192 rpy=0 0 0
